Commit message: Rename Python package to uiabot_mini_core

File: src/my_robot_bringup/urdf/uiabot_mini.urdf (robot description, URDF)
Before this commit: robot uiabot_mini, 4 links, 3 joints
Links:
- removed link wheel_l_link
- removed link wheel_r_link
- removed link world
- added link wheel_left_link; visual mesh filename=package://uiabot_mini_description/meshes/wheel.STL
- added link wheel_right_link; visual mesh filename=package://uiabot_mini_description/meshes/wheel.STL
Joints:
- removed joint base_to_wheel_l
- removed joint base_to_wheel_r
- removed joint world_to_base
- added joint joint_wheel_left: type continuous, parent base_link, child wheel_left, origin xyz=0.00060024 -0.09875 -0.022352 rpy=0 0 0, axis 0 0 1
- added joint joint_wheel_right: type continuous, parent base_link, child wheel_right, origin xyz=0.00060024 0.09875 -0.022352 rpy=0 1.57080 0, axis 0 0 1
