Commit message: Oppdatert TF etter ny STL modell

File: src/uiabot_bringup/urdf/uiabot_mini.urdf (robot description, URDF)
Before this commit: robot uiabot_mini, 4 links, 3 joints
Links:
- added link laser; visual cylinder length=0.04 radius=0.035
Joints:
- added joint joint_laser: type fixed, parent base_link, child laser, origin xyz=-49.66e-3 0.0 166.5e-3 rpy=0 0 0
- joint joint_bno055: origin xyz=71.75e-3 58.75e-3 110.35e-3 rpy=0 0 3.14159265358979 -> xyz=-71.75e-3 -58.75e-3 110.35e-3 rpy=0 0 0
- joint joint_wheel_left: origin xyz=0.00060024 -0.09875 0.0339981720062555 rpy=-1.5707963267949 0 -3.14159265358979 -> xyz=0.00060024 0.09875 0.0339981720062555 rpy=-1.5707963267948966 0 0
- joint joint_wheel_right: axis 0 0 -1 -> 0 0 1; origin xyz=0.00060024 0.09875  0.0339981720062555  rpy=1.5707963267949 0 -3.14159265358979 -> xyz=0.00060024 -0.09875  0.0339981720062555  rpy=-1.5707963267948966 0 0
