Commit message: Added SLAM, works but need to improve fuse, tried adding NAV2, need work

File: src/uiabot_mini_description/urdf/uiabot_mini.urdf (robot description, URDF)
Before this commit: robot uiabot_mini, 5 links, 4 joints
Joints:
- joint lidar_fixed_joint: origin xyz=-0.04966 0 0.1665 rpy=0 0 0 -> xyz=-0.04966 0 0.1665 rpy=0 0 3.14159265358979

Commit message: NAV2 og slam virker, fikset endel unødvendig kode.

File: src/uiabot_mini_description/urdf/uiabot_mini.urdf (robot description, URDF)
Before this commit: robot uiabot_mini, 5 links, 4 joints
Links:
- added link base_footprint
Joints:
- added joint base_footprint_joint: type fixed, parent base_link, child base_footprint, origin xyz=0 0 0.05 rpy=0 0 0
- joint lidar_fixed_joint: origin xyz=-0.04966 0 0.1665 rpy=0 0 3.14159265358979 -> xyz=0 0 0.15 rpy=0 0 3.14159265358979

Commit message: Initial commit: workspace files and xbox controller helpers

File: src/uiabot_mini_description/urdf/uiabot_mini.urdf (robot description, URDF)
Before this commit: robot uiabot_mini, 5 links, 4 joints
Links:
- added link caster_link, mass 0.05; collision sphere radius=0.019; visual sphere radius=0.019
- link base_link: mass None -> 1.0; geometry collision box size=0.15 0.12 0.06; visual mesh filename=package://uiabot_mini_description/meshes/base_link.STL
- link bno055: mass None -> 0.001
- link lidar_link: mass None -> 0.1; geometry visual cylinder length=0.04 radius=0.03
- link wheel_l_link: mass None -> 0.1; geometry collision cylinder length=0.02 radius=0.03; visual mesh filename=package://uiabot_mini_description/meshes/wheel.STL
- link wheel_r_link: mass None -> 0.1; geometry collision cylinder length=0.02 radius=0.03; visual mesh filename=package://uiabot_mini_description/meshes/wheel.STL
Joints:
- added joint caster_joint: type fixed, parent base_link, child caster_link, origin xyz=-0.0865 0 0.02235 rpy=0 0 0
- joint wheel_l_joint: origin xyz=0.00060024 0.09875 0.0339981720062555 rpy=-1.5707963267949 0 0 -> xyz=0.006 0.09875 0.034 rpy=-1.5707963267949 0 0
- joint wheel_r_joint: origin xyz=0.00060024 -0.09875  0.0339981720062555  rpy=-1.5707963267949 0 0 -> xyz=0.006 -0.09875  0.034  rpy=-1.5707963267949 0 0

Commit message: Lagt inn stol og bord, fiksa i nav sånn at det brukes velocity polygon

File: src/uiabot_mini_description/urdf/uiabot_mini.urdf (robot description, URDF)
Before this commit: robot uiabot_mini, 6 links, 5 joints
Links:
- link base_link: mass 1.0 -> None
- link caster_link: mass 0.05 -> 1.0
- link wheel_l_link: mass 0.1 -> 1.0
- link wheel_r_link: mass 0.1 -> 1.0
Joints:
- joint lidar_fixed_joint: origin xyz=0 0 0.15 rpy=0 0 3.14159265358979 -> xyz=-0.037 0 0.213 rpy=0 0 3.14159265358979
