Commit message: Fixed gazebo package

File: src/uiabot_mini_description/urdf/uiabot_differential.xacro (robot description, xacro)
@@ -7,4 +7,29 @@
     <xacro:include filename="bno055_imu.xacro.urdf" />
     <xacro:include filename="rplidar.xacro.urdf" />
-    <xacro:include filename="uiabot_mecanum_gazebo.urdf" />
+  <!-- ========= Caster Wheel ========= -->
+  <link name="caster_link">
+    <inertial>
+      <mass value="1.0"/>
+      <inertia ixx="0.00001" ixy="0.0" ixz="0.0" iyy="0.00001" iyz="0.0" izz="0.00001"/>
+    </inertial>
+    <visual>
+      <geometry>
+        <sphere radius="0.019"/>
+      </geometry>
+      <material name="green">
+        <color rgba="0.5 0.5 0.5 1.0"/>
+      </material>
+    </visual>
+    <collision>
+      <geometry>
+        <sphere radius="0.019"/>
+      </geometry>
+      <origin xyz="0 0 0" rpy="0 0 0"/>
+    </collision>
+  </link>
+  <joint name="caster_joint" type="fixed">
+    <parent link="base_link"/>
+    <child link="caster_link"/>
+    <origin xyz="-0.0865 0 0.02235" rpy="0 0 0"/>
+  </joint>
 </robot>

File: src/uiabot_mini_description/urdf/uiabot_mecanum.xacro (robot description, xacro)
@@ -7,4 +7,3 @@
     <xacro:include filename="bno055_imu.xacro.urdf" />
     <xacro:include filename="rplidar.xacro.urdf" />
-    <xacro:include filename="uiabot_mecanum_gazebo.urdf" />
 </robot>

Commit message: Code cleanup

File: src/uiabot_mini_description/urdf/uiabot_differential.xacro (robot description, xacro)
@@ -1,5 +1,7 @@
 <?xml version="1.0"?>
 <robot xmlns:xacro="http://www.ros.org/wiki/xacro" name="uiabot_mini_wrapper">
-    <xacro:property name="wheel_radius" value="0.034"/>
+    <xacro:property name="wheel_radius" value="0.034"/>          <!--Wheel radius-->
+    <xacro:property name="wheel_separation" value="197.5e-3"/>    <!--Distance between left and right wheels-->
+    <xacro:property name="wheel_front_y" value="38.1e-3"/>       <!--Front wheel y position-->
     <xacro:include filename="base_link.xacro" />
     <xacro:include filename="wheel_link.xacro"/>
@@ -23,5 +25,5 @@
     <collision>
       <geometry>
-        <sphere radius="0.019"/>
+        <sphere radius="${wheel_radius/2}"/>
       </geometry>
       <origin xyz="0 0 0" rpy="0 0 0"/>
@@ -31,5 +33,5 @@
     <parent link="base_link"/>
     <child link="caster_link"/>
-    <origin xyz="-0.0865 0 0.02235" rpy="0 0 0"/>
+    <origin xyz="-49e-3 0 ${wheel_radius/2}" rpy="0 0 0"/>
   </joint>
 </robot>

File: src/uiabot_mini_description/urdf/uiabot_mecanum.xacro (robot description, xacro)
@@ -1,5 +1,8 @@
 <?xml version="1.0"?>
 <robot xmlns:xacro="http://www.ros.org/wiki/xacro" name="uiabot_mini_wrapper">
-    <xacro:property name="wheel_radius" value="0.03"/>
+    <xacro:property name="wheel_radius" value="30e-3"/>          <!--Wheel radius-->
+    <xacro:property name="wheel_separation" value="205e-3"/>     <!--Distance between left and right wheels-->
+    <xacro:property name="wheel_base" value="75e-3"/>            <!--Distance between front and back wheels-->
+    <xacro:property name="wheel_front_y" value="38.1e-3"/>       <!--Front wheel y position-->
     <xacro:include filename="base_link.xacro" />
     <xacro:include filename="wheel_link.xacro"/>
