Commit message: Made som changes to urdf

File: src/uiabot_mecanum/urdf/uiabot_mecanum.xacro (robot description, xacro)
@@ -2,5 +2,11 @@
 <robot xmlns:xacro="http://www.ros.org/wiki/xacro" name="uiabot_mini_wrapper">
     <!-- <xacro:include filename="test.xacro.urdf" /> -->
-    <xacro:include filename="uiabot_mecanum.xacro.urdf" />
+    <xacro:property name="wheel_radius" value="0.03"/>   <!-- meters -->
+    <xacro:include filename="base_link.xacro" />
+    <xacro:include filename="wheel_link.xacro"/>
+    <xacro:include filename="mecanum_wheels.xacro.urdf" />
+    <xacro:include filename="bno055_lidar.xacro.urdf" />
+    <xacro:include filename="rplidar.xacro.urdf" />
+    <!-- <xacro:include filename="uiabot_mecanum.xacro.urdf.old" /> -->
     <xacro:include filename="uiabot_mecanum_gazebo.urdf" />
 </robot>
