Commit message: Implemented mecanum in bringup and serial. Fixed typo in urdf and added a nav2 mecanum parameter file

File: src/uiabot_mecanum/urdf/rplidar.xacro.urdf (robot description, URDF)
Before this commit: robot None, 1 links, 1 joints
Joints:
- joint lidar_fixed_joint: origin xyz=${lidar_x} ${lidar_y} ${lidar_z + wheel_radius} rpy=0 0 0 -> xyz=${lidar_x} ${lidar_y} ${lidar_z + wheel_radius} rpy=0 0 ${pi}

File: src/uiabot_mecanum/urdf/uiabot_mecanum.xacro (robot description, xacro)
@@ -6,5 +6,5 @@
     <xacro:include filename="wheel_link.xacro"/>
     <xacro:include filename="mecanum_wheels.xacro.urdf" />
-    <xacro:include filename="bno055_lidar.xacro.urdf" />
+    <xacro:include filename="bno055_imu.xacro.urdf" />
     <xacro:include filename="rplidar.xacro.urdf" />
     <!-- <xacro:include filename="uiabot_mecanum.xacro.urdf.old" /> -->
