Commit message: Added some more macros

File: src/uiabot_mecanum/urdf/bno055_imu.xacro.urdf (robot description, URDF)
Before this commit: robot None, 1 links, 1 joints
Links:
- link bno055: mass 0.001 -> ${imu_mass}

File: src/uiabot_mecanum/urdf/uiabot_mecanum.xacro (robot description, xacro)
@@ -1,6 +1,5 @@
 <?xml version="1.0"?>
 <robot xmlns:xacro="http://www.ros.org/wiki/xacro" name="uiabot_mini_wrapper">
-    <!-- <xacro:include filename="test.xacro.urdf" /> -->
-    <xacro:property name="wheel_radius" value="0.03"/>   <!-- meters -->
+    <xacro:property name="wheel_radius" value="0.03"/>
     <xacro:include filename="base_link.xacro" />
     <xacro:include filename="wheel_link.xacro"/>
@@ -8,5 +7,4 @@
     <xacro:include filename="bno055_imu.xacro.urdf" />
     <xacro:include filename="rplidar.xacro.urdf" />
-    <!-- <xacro:include filename="uiabot_mecanum.xacro.urdf.old" /> -->
     <xacro:include filename="uiabot_mecanum_gazebo.urdf" />
 </robot>

File: src/uiabot_mecanum/urdf/wheel_link.xacro (robot description, xacro)
@@ -19,12 +19,12 @@
           <mesh filename="${link_mesh}"/>
         </geometry>
-        <material name="front_left_wheel_material">
+        <material name="purple">
           <color rgba="0.5 0.0 0.5 1.0"/>
         </material>
       </visual>
       <inertial>
-        <mass value="0.5"/>
-        <inertia ixx="1e-6" ixy="0.0" ixz="0.0"
-                 iyy="1e-6" iyz="0.0" izz="1e-6"/>
+        <mass value="${wheel_mass}"/>
+        <inertia ixx="${wheel_ixx}" ixy="${wheel_ixy}" ixz="${wheel_ixz}"
+                 iyy="${wheel_iyy}" iyz="${wheel_iyz}" izz="${wheel_izz}"/>
       </inertial>
     </link>
